File: HW-Board/Negative regulation.sch (KiCad schematic (older format))
At the start: 29 parts, among them Q3 SI4436, U10 AD5245, U14 INA219POS, U16 INA2189IDR, U17 INA2189IDR, U9 MCP4725

Commit message: PDF sync
Parts:
- C28, C34: footprint (none) -> Capacitor_SMD:C_0805_2012Metric_Pad1.15x1.40mm_HandSolder
- JP4: footprint (none) -> Jumper:SolderJumper-2_P1.3mm_Open_TrianglePad1.0x1.5mm
Changed lines of the file:
@@
 F 0 "C34" H 8242 4046 50  0000 L CNN
 F 1 "1n" H 8242 3955 50  0000 L CNN
-F 2 "" H 8150 4000 50  0001 C CNN
+F 2 "Capacitor_SMD:C_0805_2012Metric_Pad1.15x1.40mm_HandSolder" H 8150 4000 50  0001 C CNN
 F 3 "~" H 8150 4000 50  0001 C CNN
 	1    8150 4000
@@
 F 0 "C28" H 3992 2696 50  0000 L CNN
 F 1 "100n50V" H 3992 2605 50  0000 L CNN
-F 2 "" H 3900 2650 50  0001 C CNN
+F 2 "Capacitor_SMD:C_0805_2012Metric_Pad1.15x1.40mm_HandSolder" H 3900 2650 50  0001 C CNN
 F 3 "~" H 3900 2650 50  0001 C CNN
 	1    3900 2650
@@
 F 0 "JP4" H 2750 3314 50  0000 C CNN
 F 1 "Jumper" H 2750 3223 50  0000 C CNN
-F 2 "" H 2750 3050 50  0001 C CNN
+F 2 "Jumper:SolderJumper-2_P1.3mm_Open_TrianglePad1.0x1.5mm" H 2750 3050 50  0001 C CNN
 F 3 "~" H 2750 3050 50  0001 C CNN
 	1    2750 3050
